File: pcb/avrdmx.sch (EAGLE design)
At the start: 15 parts, among them U1 ARDUINO_SHIELDLABEL

Commit message: schematic changes from a long time ago, not sure if they're good
Parts:
- removed INVERTER: 7404N, 74xx-us:7404N
- removed R1, R2, R3, R4: 10K, SparkFun-Resistors:RESISTORPTH-1/4W
- removed SW1: (no value), special:SW_DIP-4
- removed TAIL1, TAIL2, TAIL3, TAIL4: (no value), SparkFun-Connectors:M03-SCREW-5MM
- added DRIVER5: 75176AP, 751xx:75176AP
- added IR1: IR IN, pinhead:PINHD-1X3
- added OUT1, OUT2, OUT3, OUT4: NC5FAV, avrdmx:NC5FAV
- added TAIL5: DMX IN, SparkFun-Connectors:M03-SCREW-5MM
Connections:
- removed net N$17: DRIVER2.A, TAIL2.1
- removed net N$18: DRIVER2.B, TAIL2.2
- removed net N$19: DRIVER3.A, TAIL3.1
- removed net N$20: DRIVER3.B, TAIL3.2
- removed net N$21: DRIVER4.A, TAIL4.1
- removed net N$22: DRIVER4.B, TAIL4.2
- new net N$15: DRIVER4.A, OUT4.3
- new net N$6: DRIVER5.A, TAIL5.1
- net GND: now also DRIVER1.R, DRIVER2.R, DRIVER3.R, DRIVER4.R, DRIVER5.!RE, DRIVER5.D, DRIVER5.DE, DRIVER5.GND, IR1.2, OUT1.1, OUT2.1, OUT3.1, OUT4.1, TAIL5.3; no longer R1.1, R2.1, R3.1, R4.1, TAIL1.3, TAIL2.3, TAIL3.3, TAIL4.3
- net N$1: no longer DRIVER1.R
- net N$10: now also OUT1.3; no longer TAIL1.1
- net N$11: now also DRIVER2.B, OUT2.2; no longer DRIVER1.!RE, INVERTERA.I, R1.2, SW1.1
- net N$12: now also DRIVER2.A, OUT2.3; no longer DRIVER2.!RE, INVERTERB.I, R2.2, SW1.2
- net N$13: now also DRIVER3.B, OUT3.2; no longer DRIVER3.!RE, INVERTERC.I, R3.2, SW1.3
- net N$14: now also DRIVER3.A, OUT3.3; no longer DRIVER4.!RE, INVERTERD.I, R4.2, SW1.4
- net N$16: now also DRIVER4.B, OUT4.2; no longer DRIVER1.B, TAIL1.2
- net N$2: no longer DRIVER2.R
- net N$3: no longer DRIVER3.R
- net N$4: no longer DRIVER4.R
- net N$5: now also IR1.1, U1.D7; no longer DRIVER4.DE, INVERTERD.O
- net N$7: now also DRIVER5.B, TAIL5.2; no longer DRIVER3.DE, INVERTERC.O
- net N$8: now also DRIVER1.B, OUT1.2; no longer DRIVER2.DE, INVERTERB.O
- net N$9: now also DRIVER5.R, U1.RX; no longer DRIVER1.DE, INVERTERA.O
- net VCC: now also DRIVER1.!RE, DRIVER1.DE, DRIVER2.!RE, DRIVER2.DE, DRIVER3.!RE, DRIVER3.DE, DRIVER4.!RE, DRIVER4.DE, DRIVER5.VCC, IR1.3; no longer SW1.5, SW1.6, SW1.7, SW1.8

Commit message: finish PCB rev3
Parts:
- removed OUT1, OUT2, OUT3, OUT4: NC5FAV, avrdmx:NC5FAV
- removed TAIL5: DMX IN, SparkFun-Connectors:M03-SCREW-5MM
- added U$1, U$2, U$3, U$4, U$5: B3P-VH, avrdmx:B3P-VH
Connections:
- net GND: now also U$1.G, U$2.G, U$3.G, U$4.G, U$5.A; no longer OUT1.1, OUT2.1, OUT3.1, OUT4.1, TAIL5.3
- net N$10: now also U$1.A; no longer OUT1.3
- net N$11: now also U$2.B; no longer OUT2.2
- net N$12: now also U$2.A; no longer OUT2.3
- net N$13: now also U$3.B; no longer OUT3.2
- net N$14: now also U$3.A; no longer OUT3.3
- net N$15: now also U$4.A; no longer OUT4.3
- net N$16: now also U$4.B; no longer OUT4.2
- net N$5: now also U1.A0; no longer U1.D7
- net N$6: now also U$5.G; no longer TAIL5.1
- net N$7: now also U$5.B; no longer TAIL5.2
- net N$8: now also U$1.B; no longer OUT1.2
Changed lines of the file:
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@@
 <part name="P+10" library="supply1" deviceset="VCC" device=""/>
 <part name="GND2" library="supply1" deviceset="GND" device=""/>
-<part name="U$1" library="avrdmx" deviceset="SN75176" device=""/>
-<part name="U$2" library="avrdmx" deviceset="SN75176" device=""/>
-<part name="U$3" library="avrdmx" deviceset="SN75176" device=""/>
-<part name="U$4" library="avrdmx" deviceset="SN75176" device=""/>
-<part name="U$5" library="avrdmx" deviceset="SN75176" device=""/>
-<part name="U$6" library="avrdmx" deviceset="SN75176" device=""/>
-<part name="U$7" library="avrdmx" deviceset="SN75176" device=""/>
-<part name="U$8" library="avrdmx" deviceset="SN75176" device=""/>
 <part name="DRIVER5" library="751xx" deviceset="75176A" device="P"/>
 <part name="P+11" library="supply1" deviceset="VCC" device=""/>
 <part name="GND6" library="supply1" deviceset="GND" device=""/>
-<part name="TAIL5" library="SparkFun-Connectors" deviceset="M03" device="-SCREW-5MM" value="DMX IN"/>
 <part name="IR1" library="pinhead" deviceset="PINHD-1X3" device="" value="IR IN"/>
 <part name="GND7" library="supply1" deviceset="GND" device=""/>
@@
 <part name="GND10" library="supply1" deviceset="GND" device=""/>
 <part name="GND11" library="supply1" deviceset="GND" device=""/>
-<part name="OUT1" library="avrdmx" deviceset="NC5FAV" device=""/>
-<part name="OUT2" library="avrdmx" deviceset="NC5FAV" device=""/>
-<part name="OUT3" library="avrdmx" deviceset="NC5FAV" device=""/>
-<part name="OUT4" library="avrdmx" deviceset="NC5FAV" device=""/>
+<part name="U$1" library="avrdmx" deviceset="B3P-VH" device=""/>
+<part name="U$2" library="avrdmx" deviceset="B3P-VH" device=""/>
+<part name="U$3" library="avrdmx" deviceset="B3P-VH" device=""/>
+<part name="U$4" library="avrdmx" deviceset="B3P-VH" device=""/>
+<part name="U$5" library="avrdmx" deviceset="B3P-VH" device=""/>
 </parts>
 <sheets>
@@
 <instance part="P+11" gate="VCC" x="10.16" y="38.1"/>
 <instance part="GND6" gate="1" x="-22.86" y="7.62"/>
-<instance part="TAIL5" gate="G$1" x="20.32" y="25.4" rot="R180"/>
 <instance part="IR1" gate="A" x="33.02" y="96.52"/>
 <instance part="GND7" gate="1" x="27.94" y="81.28"/>
@@
 <instance part="GND10" gate="1" x="38.1" y="25.4"/>
 <instance part="GND11" gate="1" x="38.1" y="0"/>
-<instance part="OUT1" gate="G$1" x="83.82" y="78.74"/>
-<instance part="OUT2" gate="G$1" x="83.82" y="53.34"/>
-<instance part="OUT3" gate="G$1" x="83.82" y="27.94"/>
-<instance part="OUT4" gate="G$1" x="83.82" y="2.54"/>
+<instance part="U$1" gate="G$1" x="83.82" y="81.28"/>
+<instance part="U$2" gate="G$1" x="83.82" y="55.88"/>
+<instance part="U$3" gate="G$1" x="83.82" y="30.48"/>
+<instance part="U$4" gate="G$1" x="83.82" y="5.08"/>
+<instance part="U$5" gate="G$1" x="20.32" y="25.4"/>
 </instances>
 <busses>
@@
 <wire x1="7.62" y1="12.7" x2="-22.86" y2="12.7" width="0.1524" layer="91"/>
 <junction x="-22.86" y="12.7"/>
-<pinref part="TAIL5" gate="G$1" pin="3"/>
 <wire x1="12.7" y1="22.86" x2="12.7" y2="17.78" width="0.1524" layer="91"/>
 <wire x1="12.7" y1="17.78" x2="7.62" y2="17.78" width="0.1524" layer="91"/>
@@
 <wire x1="-17.78" y1="30.48" x2="-22.86" y2="30.48" width="0.1524" layer="91"/>
 <junction x="-22.86" y="30.48"/>
+<pinref part="U$5" gate="G$1" pin="A"/>
 </segment>
 <segment>
@@
 <wire x1="93.98" y1="68.58" x2="93.98" y2="88.9" width="0.1524" layer="91"/>
 <wire x1="93.98" y1="88.9" x2="76.2" y2="88.9" width="0.1524" layer="91"/>
-<pinref part="OUT1" gate="G$1" pin="1"/>
 <wire x1="76.2" y1="88.9" x2="76.2" y2="83.82" width="0.1524" layer="91"/>
 <wire x1="93.98" y1="63.5" x2="76.2" y2="63.5" width="0.1524" layer="91"/>
 <junction x="93.98" y="63.5"/>
-<pinref part="OUT2" gate="G$1" pin="1"/>
 <wire x1="76.2" y1="63.5" x2="76.2" y2="58.42" width="0.1524" layer="91"/>
 <wire x1="93.98" y1="38.1" x2="76.2" y2="38.1" width="0.1524" layer="91"/>
 <junction x="93.98" y="38.1"/>
-<pinref part="OUT3" gate="G$1" pin="1"/>
 <wire x1="76.2" y1="38.1" x2="76.2" y2="33.02" width="0.1524" layer="91"/>
 <wire x1="93.98" y1="12.7" x2="76.2" y2="12.7" width="0.1524" layer="91"/>
 <junction x="93.98" y="12.7"/>
-<pinref part="OUT4" gate="G$1" pin="1"/>
 <wire x1="76.2" y1="12.7" x2="76.2" y2="7.62" width="0.1524" layer="91"/>
 <pinref part="DRIVER3" gate="G$1" pin="GND"/>
@@
 <wire x1="73.66" y1="68.58" x2="93.98" y2="68.58" width="0.1524" layer="91"/>
 <junction x="93.98" y="68.58"/>
+<pinref part="U$1" gate="G$1" pin="G"/>
+<pinref part="U$2" gate="G$1" pin="G"/>
+<pinref part="U$3" gate="G$1" pin="G"/>
+<pinref part="U$4" gate="G$1" pin="G"/>
 </segment>
 </net>
@@
 <segment>
 <pinref part="DRIVER5" gate="G$1" pin="A"/>
-<pinref part="TAIL5" gate="G$1" pin="1"/>
 <wire x1="7.62" y1="27.94" x2="12.7" y2="27.94" width="0.1524" layer="91"/>
+<pinref part="U$5" gate="G$1" pin="G"/>
 </segment>
 </net>
@@
 <segment>
 <pinref part="DRIVER5" gate="G$1" pin="B"/>
-<pinref part="TAIL5" gate="G$1" pin="2"/>
 <wire x1="7.62" y1="25.4" x2="12.7" y2="25.4" width="0.1524" layer="91"/>
+<pinref part="U$5" gate="G$1" pin="B"/>
 </segment>
 </net>
@@
 <segment>
 <pinref part="IR1" gate="A" pin="1"/>
-<wire x1="30.48" y1="99.06" x2="22.86" y2="99.06" width="0.1524" layer="91"/>
-<wire x1="22.86" y1="99.06" x2="22.86" y2="68.58" width="0.1524" layer="91"/>
-<pinref part="U1" gate="G$1" pin="D7"/>
-<wire x1="22.86" y1="68.58" x2="17.78" y2="68.58" width="0.1524" layer="91"/>
+<wire x1="30.48" y1="99.06" x2="-10.16" y2="99.06" width="0.1524" layer="91"/>
+<wire x1="-10.16" y1="99.06" x2="-10.16" y2="88.9" width="0.1524" layer="91"/>
+<pinref part="U1" gate="G$1" pin="A0"/>
+<wire x1="-10.16" y1="88.9" x2="-7.62" y2="88.9" width="0.1524" layer="91"/>
 </segment>
 </net>
@@
 <segment>
 <pinref part="DRIVER1" gate="G$1" pin="B"/>
-<pinref part="OUT1" gate="G$1" pin="2"/>
 <wire x1="68.58" y1="81.28" x2="76.2" y2="81.28" width="0.1524" layer="91"/>
+<pinref part="U$1" gate="G$1" pin="B"/>
 </segment>
 </net>
@@
 <wire x1="68.58" y1="83.82" x2="71.12" y2="83.82" width="0.1524" layer="91"/>
 <wire x1="71.12" y1="83.82" x2="71.12" y2="78.74" width="0.1524" layer="91"/>
-<pinref part="OUT1" gate="G$1" pin="3"/>
 <wire x1="71.12" y1="78.74" x2="76.2" y2="78.74" width="0.1524" layer="91"/>
+<pinref part="U$1" gate="G$1" pin="A"/>
 </segment>
 </net>
@@
 <segment>
 <pinref part="DRIVER2" gate="G$1" pin="B"/>
-<pinref part="OUT2" gate="G$1" pin="2"/>
 <wire x1="68.58" y1="55.88" x2="76.2" y2="55.88" width="0.1524" layer="91"/>
+<pinref part="U$2" gate="G$1" pin="B"/>
 </segment>
 </net>
@@
 <wire x1="68.58" y1="58.42" x2="71.12" y2="58.42" width="0.1524" layer="91"/>
 <wire x1="71.12" y1="58.42" x2="71.12" y2="53.34" width="0.1524" layer="91"/>
-<pinref part="OUT2" gate="G$1" pin="3"/>
 <wire x1="71.12" y1="53.34" x2="76.2" y2="53.34" width="0.1524" layer="91"/>
+<pinref part="U$2" gate="G$1" pin="A"/>
 </segment>
 </net>
@@
 <segment>
 <pinref part="DRIVER3" gate="G$1" pin="B"/>
-<pinref part="OUT3" gate="G$1" pin="2"/>
 <wire x1="68.58" y1="30.48" x2="76.2" y2="30.48" width="0.1524" layer="91"/>
+<pinref part="U$3" gate="G$1" pin="B"/>
 </segment>
 </net>
@@
 <wire x1="68.58" y1="33.02" x2="71.12" y2="33.02" width="0.1524" layer="91"/>
 <wire x1="71.12" y1="33.02" x2="71.12" y2="27.94" width="0.1524" layer="91"/>
-<pinref part="OUT3" gate="G$1" pin="3"/>
 <wire x1="71.12" y1="27.94" x2="76.2" y2="27.94" width="0.1524" layer="91"/>
+<pinref part="U$3" gate="G$1" pin="A"/>
 </segment>
 </net>
@@
 <wire x1="68.58" y1="7.62" x2="71.12" y2="7.62" width="0.1524" layer="91"/>
 <wire x1="71.12" y1="7.62" x2="71.12" y2="2.54" width="0.1524" layer="91"/>
-<pinref part="OUT4" gate="G$1" pin="3"/>
 <wire x1="71.12" y1="2.54" x2="76.2" y2="2.54" width="0.1524" layer="91"/>
+<pinref part="U$4" gate="G$1" pin="A"/>
 </segment>
 </net>
@@
 <segment>
 <pinref part="DRIVER4" gate="G$1" pin="B"/>
-<pinref part="OUT4" gate="G$1" pin="2"/>
 <wire x1="68.58" y1="5.08" x2="76.2" y2="5.08" width="0.1524" layer="91"/>
-</segment>
-</net>
+<pinref part="U$4" gate="G$1" pin="B"/>
+</segment>
+</net>

Commit message: PCB rev4 - fixes:  - larger holes for DMX cable headers  - fix receiver driver wiring  - better labels
Parts:
- ANALOG_IN: value IR IN -> ANALOG IN
- renumbered DRIVER5 to DRIVER_IN, IR1 to ANALOG_IN, U$1 to DMX1, U$2 to DMX2, U$3 to DMX3, U$4 to DMX4, U$5 to DMX_IN
Connections:
- removed net N$6: DMX_IN.G, DRIVER_IN.A
- new net N$17: DMX_IN.A, DRIVER_IN.A
- net GND: now also DMX_IN.G; no longer DMX_IN.A
Changed lines of the file:
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@@
 <?xml version="1.0" encoding="utf-8"?>
 <!DOCTYPE eagle SYSTEM "eagle.dtd">
-<eagle version="6.4">
+<eagle version="6.5.0">
 <drawing>
 <settings>
@@
 <part name="P+10" library="supply1" deviceset="VCC" device=""/>
 <part name="GND2" library="supply1" deviceset="GND" device=""/>
-<part name="DRIVER5" library="751xx" deviceset="75176A" device="P"/>
+<part name="DRIVER_IN" library="751xx" deviceset="75176A" device="P"/>
 <part name="P+11" library="supply1" deviceset="VCC" device=""/>
 <part name="GND6" library="supply1" deviceset="GND" device=""/>
-<part name="IR1" library="pinhead" deviceset="PINHD-1X3" device="" value="IR IN"/>
+<part name="ANALOG_IN" library="pinhead" deviceset="PINHD-1X3" device="" value="ANALOG IN"/>
 <part name="GND7" library="supply1" deviceset="GND" device=""/>
 <part name="GND8" library="supply1" deviceset="GND" device=""/>
@@
 <part name="GND10" library="supply1" deviceset="GND" device=""/>
 <part name="GND11" library="supply1" deviceset="GND" device=""/>
-<part name="U$1" library="avrdmx" deviceset="B3P-VH" device=""/>
-<part name="U$2" library="avrdmx" deviceset="B3P-VH" device=""/>
-<part name="U$3" library="avrdmx" deviceset="B3P-VH" device=""/>
-<part name="U$4" library="avrdmx" deviceset="B3P-VH" device=""/>
-<part name="U$5" library="avrdmx" deviceset="B3P-VH" device=""/>
+<part name="DMX1" library="avrdmx" deviceset="B3P-VH" device=""/>
+<part name="DMX2" library="avrdmx" deviceset="B3P-VH" device=""/>
+<part name="DMX3" library="avrdmx" deviceset="B3P-VH" device=""/>
+<part name="DMX4" library="avrdmx" deviceset="B3P-VH" device=""/>
+<part name="DMX_IN" library="avrdmx" deviceset="B3P-VH" device=""/>
 </parts>
 <sheets>
@@
 <instance part="P+10" gate="VCC" x="71.12" y="17.78"/>
 <instance part="GND2" gate="1" x="71.12" y="-10.16"/>
-<instance part="DRIVER5" gate="G$1" x="-5.08" y="27.94"/>
+<instance part="DRIVER_IN" gate="G$1" x="-5.08" y="27.94"/>
 <instance part="P+11" gate="VCC" x="10.16" y="38.1"/>
 <instance part="GND6" gate="1" x="-22.86" y="7.62"/>
-<instance part="IR1" gate="A" x="33.02" y="96.52"/>
+<instance part="ANALOG_IN" gate="A" x="33.02" y="96.52"/>
 <instance part="GND7" gate="1" x="27.94" y="81.28"/>
 <instance part="GND8" gate="1" x="38.1" y="76.2"/>
@@
 <instance part="GND10" gate="1" x="38.1" y="25.4"/>
 <instance part="GND11" gate="1" x="38.1" y="0"/>
-<instance part="U$1" gate="G$1" x="83.82" y="81.28"/>
-<instance part="U$2" gate="G$1" x="83.82" y="55.88"/>
-<instance part="U$3" gate="G$1" x="83.82" y="30.48"/>
-<instance part="U$4" gate="G$1" x="83.82" y="5.08"/>
-<instance part="U$5" gate="G$1" x="20.32" y="25.4"/>
+<instance part="DMX1" gate="G$1" x="83.82" y="81.28"/>
+<instance part="DMX2" gate="G$1" x="83.82" y="55.88"/>
+<instance part="DMX3" gate="G$1" x="83.82" y="30.48"/>
+<instance part="DMX4" gate="G$1" x="83.82" y="5.08"/>
+<instance part="DMX_IN" gate="G$1" x="20.32" y="25.4"/>
 </instances>
 <busses>
@@
 </segment>
 <segment>
-<pinref part="DRIVER5" gate="G$1" pin="!RE"/>
+<pinref part="DRIVER_IN" gate="G$1" pin="!RE"/>
 <wire x1="-17.78" y1="25.4" x2="-22.86" y2="25.4" width="0.1524" layer="91"/>
 <pinref part="GND6" gate="1" pin="GND"/>
 <wire x1="-22.86" y1="25.4" x2="-22.86" y2="12.7" width="0.1524" layer="91"/>
-<pinref part="DRIVER5" gate="G$1" pin="DE"/>
+<pinref part="DRIVER_IN" gate="G$1" pin="DE"/>
 <wire x1="-22.86" y1="12.7" x2="-22.86" y2="10.16" width="0.1524" layer="91"/>
 <wire x1="-17.78" y1="33.02" x2="-22.86" y2="33.02" width="0.1524" layer="91"/>
 <wire x1="-22.86" y1="33.02" x2="-22.86" y2="30.48" width="0.1524" layer="91"/>
 <junction x="-22.86" y="25.4"/>
-<pinref part="DRIVER5" gate="G$1" pin="GND"/>
+<pinref part="DRIVER_IN" gate="G$1" pin="GND"/>
 <wire x1="-22.86" y1="30.48" x2="-22.86" y2="25.4" width="0.1524" layer="91"/>
-<wire x1="7.62" y1="20.32" x2="7.62" y2="17.78" width="0.1524" layer="91"/>
-<wire x1="7.62" y1="17.78" x2="7.62" y2="12.7" width="0.1524" layer="91"/>
+<wire x1="7.62" y1="20.32" x2="7.62" y2="12.7" width="0.1524" layer="91"/>
 <wire x1="7.62" y1="12.7" x2="-22.86" y2="12.7" width="0.1524" layer="91"/>
 <junction x="-22.86" y="12.7"/>
-<wire x1="12.7" y1="22.86" x2="12.7" y2="17.78" width="0.1524" layer="91"/>
-<wire x1="12.7" y1="17.78" x2="7.62" y2="17.78" width="0.1524" layer="91"/>
-<junction x="7.62" y="17.78"/>
-<pinref part="DRIVER5" gate="G$1" pin="D"/>
+<pinref part="DRIVER_IN" gate="G$1" pin="D"/>
 <wire x1="-17.78" y1="30.48" x2="-22.86" y2="30.48" width="0.1524" layer="91"/>
 <junction x="-22.86" y="30.48"/>
-<pinref part="U$5" gate="G$1" pin="A"/>
-</segment>
-<segment>
-<pinref part="IR1" gate="A" pin="2"/>
+<pinref part="DMX_IN" gate="G$1" pin="G"/>
+<wire x1="12.7" y1="27.94" x2="12.7" y2="33.02" width="0.1524" layer="91"/>
+<wire x1="12.7" y1="33.02" x2="25.4" y2="33.02" width="0.1524" layer="91"/>
+<wire x1="25.4" y1="33.02" x2="25.4" y2="12.7" width="0.1524" layer="91"/>
+<wire x1="25.4" y1="12.7" x2="7.62" y2="12.7" width="0.1524" layer="91"/>
+<junction x="7.62" y="12.7"/>
+</segment>
+<segment>
+<pinref part="ANALOG_IN" gate="A" pin="2"/>
 <pinref part="GND7" gate="1" pin="GND"/>
 <wire x1="30.48" y1="96.52" x2="27.94" y2="96.52" width="0.1524" layer="91"/>
@@
 <wire x1="73.66" y1="68.58" x2="93.98" y2="68.58" width="0.1524" layer="91"/>
 <junction x="93.98" y="68.58"/>
-<pinref part="U$1" gate="G$1" pin="G"/>
-<pinref part="U$2" gate="G$1" pin="G"/>
-<pinref part="U$3" gate="G$1" pin="G"/>
-<pinref part="U$4" gate="G$1" pin="G"/>
+<pinref part="DMX1" gate="G$1" pin="G"/>
+<pinref part="DMX2" gate="G$1" pin="G"/>
+<pinref part="DMX3" gate="G$1" pin="G"/>
+<pinref part="DMX4" gate="G$1" pin="G"/>
 </segment>
 </net>
@@
 <wire x1="40.64" y1="81.28" x2="40.64" y2="88.9" width="0.1524" layer="91"/>
 <junction x="40.64" y="88.9"/>
-<pinref part="IR1" gate="A" pin="3"/>
+<pinref part="ANALOG_IN" gate="A" pin="3"/>
 <wire x1="30.48" y1="93.98" x2="30.48" y2="88.9" width="0.1524" layer="91"/>
 <wire x1="30.48" y1="88.9" x2="40.64" y2="88.9" width="0.1524" layer="91"/>
@@
 <pinref part="P+11" gate="VCC" pin="VCC"/>
 <wire x1="10.16" y1="35.56" x2="10.16" y2="33.02" width="0.1524" layer="91"/>
-<pinref part="DRIVER5" gate="G$1" pin="VCC"/>
+<pinref part="DRIVER_IN" gate="G$1" pin="VCC"/>
 <wire x1="10.16" y1="33.02" x2="7.62" y2="33.02" width="0.1524" layer="91"/>
 </segment>
 </net>
-<net name="N$6" class="0">
-<segment>
-<pinref part="DRIVER5" gate="G$1" pin="A"/>
-<wire x1="7.62" y1="27.94" x2="12.7" y2="27.94" width="0.1524" layer="91"/>
-<pinref part="U$5" gate="G$1" pin="G"/>
-</segment>
-</net>
-<net name="N$7" class="0">
-<segment>
-<pinref part="DRIVER5" gate="G$1" pin="B"/>
-<wire x1="7.62" y1="25.4" x2="12.7" y2="25.4" width="0.1524" layer="91"/>
-<pinref part="U$5" gate="G$1" pin="B"/>
-</segment>
-</net>
 <net name="N$9" class="0">
 <segment>
-<pinref part="DRIVER5" gate="G$1" pin="R"/>
+<pinref part="DRIVER_IN" gate="G$1" pin="R"/>
 <wire x1="-17.78" y1="22.86" x2="-45.72" y2="22.86" width="0.1524" layer="91"/>
 <wire x1="-45.72" y1="22.86" x2="-45.72" y2="96.52" width="0.1524" layer="91"/>
@@
 <net name="N$5" class="0">
 <segment>
-<pinref part="IR1" gate="A" pin="1"/>
+<pinref part="ANALOG_IN" gate="A" pin="1"/>
 <wire x1="30.48" y1="99.06" x2="-10.16" y2="99.06" width="0.1524" layer="91"/>
 <wire x1="-10.16" y1="99.06" x2="-10.16" y2="88.9" width="0.1524" layer="91"/>
@@
 <pinref part="DRIVER1" gate="G$1" pin="B"/>
 <wire x1="68.58" y1="81.28" x2="76.2" y2="81.28" width="0.1524" layer="91"/>
-<pinref part="U$1" gate="G$1" pin="B"/>
+<pinref part="DMX1" gate="G$1" pin="B"/>
 </segment>
 </net>
@@
 <wire x1="71.12" y1="83.82" x2="71.12" y2="78.74" width="0.1524" layer="91"/>
 <wire x1="71.12" y1="78.74" x2="76.2" y2="78.74" width="0.1524" layer="91"/>
-<pinref part="U$1" gate="G$1" pin="A"/>
+<pinref part="DMX1" gate="G$1" pin="A"/>
 </segment>
 </net>
@@
 <pinref part="DRIVER2" gate="G$1" pin="B"/>
 <wire x1="68.58" y1="55.88" x2="76.2" y2="55.88" width="0.1524" layer="91"/>
-<pinref part="U$2" gate="G$1" pin="B"/>
+<pinref part="DMX2" gate="G$1" pin="B"/>
 </segment>
 </net>
@@
 <wire x1="71.12" y1="58.42" x2="71.12" y2="53.34" width="0.1524" layer="91"/>
 <wire x1="71.12" y1="53.34" x2="76.2" y2="53.34" width="0.1524" layer="91"/>
-<pinref part="U$2" gate="G$1" pin="A"/>
+<pinref part="DMX2" gate="G$1" pin="A"/>
 </segment>
 </net>
@@
 <pinref part="DRIVER3" gate="G$1" pin="B"/>
 <wire x1="68.58" y1="30.48" x2="76.2" y2="30.48" width="0.1524" layer="91"/>
-<pinref part="U$3" gate="G$1" pin="B"/>
+<pinref part="DMX3" gate="G$1" pin="B"/>
 </segment>
 </net>
@@
 <wire x1="71.12" y1="33.02" x2="71.12" y2="27.94" width="0.1524" layer="91"/>
 <wire x1="71.12" y1="27.94" x2="76.2" y2="27.94" width="0.1524" layer="91"/>
-<pinref part="U$3" gate="G$1" pin="A"/>
+<pinref part="DMX3" gate="G$1" pin="A"/>
 </segment>
 </net>
@@
 <wire x1="71.12" y1="7.62" x2="71.12" y2="2.54" width="0.1524" layer="91"/>
 <wire x1="71.12" y1="2.54" x2="76.2" y2="2.54" width="0.1524" layer="91"/>
-<pinref part="U$4" gate="G$1" pin="A"/>
+<pinref part="DMX4" gate="G$1" pin="A"/>
 </segment>
 </net>
@@
 <pinref part="DRIVER4" gate="G$1" pin="B"/>
 <wire x1="68.58" y1="5.08" x2="76.2" y2="5.08" width="0.1524" layer="91"/>
-<pinref part="U$4" gate="G$1" pin="B"/>
-</segment>
-</net>
+<pinref part="DMX4" gate="G$1" pin="B"/>
+</segment>
+</net>
+<net name="N$7" class="0">
+<segment>
+<pinref part="DMX_IN" gate="G$1" pin="B"/>
+<pinref part="DRIVER_IN" gate="G$1" pin="B"/>
+<wire x1="12.7" y1="25.4" x2="7.62" y2="25.4" width="0.1524" layer="91"/>
+</segment>
+</net>
+<net name="N$17" class="0">
+<segment>
+<pinref part="DMX_IN" gate="G$1" pin="A"/>
+<wire x1="12.7" y1="22.86" x2="10.16" y2="22.86" width="0.1524" layer="91"/>
+<wire x1="10.16" y1="22.86" x2="10.16" y2="27.94" width="0.1524" layer="91"/>
+<pinref part="DRIVER_IN" gate="G$1" pin="A"/>
+<wire x1="10.16" y1="27.94" x2="7.62" y2="27.94" width="0.1524" layer="91"/>
+</segment>
+</net>
