File: avrdmxsmt/avrdmxsmt.brd (EAGLE design)
At the start: 44.1 x 33 mm, 27 parts, among them J1 AVR_SPI_PRG_6PTH, Q1 16MHz

Commit message: SMT board cleanup
Parts:
- added HWB: HWB, SparkFun-Passives:1X02
- moved R1 9.60 mm to (25.4, 24.6), turned to 0 degrees
- moved C7 0.51 mm to (35.1, 2.29), turned to 90 degrees
- moved R3 0.25 mm to (1.52, 25.9), turned to 90 degrees
- moved C5 0.25 mm to (2.79, 23.0)
- turned R2 to 90 degrees
- renumbered D1 to RED, D2 to GREEN, D3 to YELLOW, F1 to FUSE, SN1 to SN75174
Connections:
- new net N$25: AVR.33, HWB.2
- net GND: now also HWB.1; no longer AVR.33
Routing:
- net VCC: track 129.1 -> 110.9 mm, vias 4 -> 3
- net GND: track 201.1 -> 217.8 mm
- net N$1: track 63.7 -> 77.5 mm
- net N$25: track 0.00 -> 12.3 mm
- net N$14: track 61.3 -> 49.6 mm
- net N$29: track 22.1 -> 32.7 mm, vias 2 -> 1
- net N$15: track 42.0 -> 50.0 mm
- net N$9: track 31.7 -> 24.0 mm
- net N$3: track 6.54 -> 13.6 mm, vias 2 -> 0
- net N$27: track 22.8 -> 27.6 mm
- net N$31: track 32.0 -> 27.6 mm, vias 1 -> 2
- net N$2: track 30.4 -> 34.3 mm
- net N$8: track 32.3 -> 35.6 mm
- net N$10: track 35.4 -> 38.7 mm
- net N$19: track 35.6 -> 38.9 mm
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Other:
- board text added: "AVR DMX rev5"
- board text removed: "AVR DMX r5"
