File: avrdmxsmt/avrdmxsmt.brd (EAGLE design)
At the start: 44.1 x 33 mm, 28 parts, among them J1 AVR_SPI_PRG_6PTH, Q1 16MHz

Commit message: surface mount PCB drill sizes, cleanup
Parts:
- moved C4 1.10 mm to (21.0, 23.4)
- moved FUSE 0.85 mm to (7.50, 24.5)
Routing:
- net N$7: track 23.0 -> 56.3 mm
- net N$1: track 77.5 -> 48.2 mm
- net VCC: track 110.9 -> 132.0 mm, vias 3 -> 5
- net GND: track 217.8 -> 208.8 mm
- net N$4: track 30.8 -> 24.0 mm
- net N$14: track 49.6 -> 45.6 mm
- net N$8: track 35.6 -> 31.9 mm
- net N$30: track 24.8 -> 27.8 mm
- net N$13: track 30.2 -> 33.2 mm
- net N$29: track 32.7 -> 30.6 mm
- net N$2: track 34.3 -> 35.5 mm
- net N$31: track 27.6 -> 28.6 mm
- net N$15: track 50.0 -> 51.0 mm
- net N$16: track 31.3 -> 32.0 mm
- net N$19: track 38.9 -> 38.2 mm
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