File: avrdmxsmt/avrdmxsmt.sch (EAGLE design)
At the start: 27 parts, among them J1 AVR_SPI_PRG_6PTH, Q1 16MHz

Commit message: SMT board cleanup
Parts:
- added HWB: HWB, SparkFun-Passives:JUMPER-2PTH
- renumbered D1 to RED, D2 to GREEN, D3 to YELLOW, F1 to FUSE, SN1 to SN75174
Connections:
- new net N$25: AVR.PE2/!HWB, HWB.2
- net GND: now also HWB.1; no longer AVR.PE2/!HWB
Other:
- moved on the sheet: C4, C5, C6, C7
